File: hardware/pcb/OpenNav_Windsensor.kicad_sch (KiCad schematic)
At the start: 9 parts, among them IC1 AS5600-ASOT, J1 Conn_01x02_Pin, U1 XIAO-ESP32-C6, U2 StpDwnE3.3-0.5, U3 SS411P, U4 DS18B20

Commit message: SMD V2
Parts:
- C3: footprint Capacitor_THT:C_Disc_D8.0mm_W5.0mm_P7.50mm -> Capacitor_SMD:C_0603_1608Metric_Pad1.08x0.95mm_HandSolder
- R1, R2: footprint Resistor_THT:R_Axial_DIN0207_L6.3mm_D2.5mm_P7.62mm_Horizontal -> Resistor_SMD:R_0603_1608Metric_Pad0.98x0.95mm_HandSolder
- U1: footprint Seeed Studio XIAO Series Library:XIAO-ESP32C6-DIP -> Seeed Studio XIAO Series Library:XIAO-ESP32C6-SMD
Changed lines of the file:
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@@
 			)
 		)
-		(property "Footprint" "Seeed Studio XIAO Series Library:XIAO-ESP32C6-DIP"
+		(property "Footprint" "Seeed Studio XIAO Series Library:XIAO-ESP32C6-SMD"
 			(at 145.288 134.112 0)
 			(effects
@@
 			)
 		)
-		(property "Footprint" "Resistor_THT:R_Axial_DIN0207_L6.3mm_D2.5mm_P7.62mm_Horizontal"
+		(property "Footprint" "Resistor_SMD:R_0603_1608Metric_Pad0.98x0.95mm_HandSolder"
 			(at 120.65 125.73 0)
 			(effects
@@
 			)
 		)
-		(property "Footprint" "Resistor_THT:R_Axial_DIN0207_L6.3mm_D2.5mm_P7.62mm_Horizontal"
+		(property "Footprint" "Resistor_SMD:R_0603_1608Metric_Pad0.98x0.95mm_HandSolder"
 			(at 118.11 125.73 0)
 			(effects
@@
 			)
 		)
-		(property "Footprint" "Capacitor_THT:C_Disc_D8.0mm_W5.0mm_P7.50mm"
+		(property "Footprint" "Capacitor_SMD:C_0603_1608Metric_Pad1.08x0.95mm_HandSolder"
 			(at 78.74 123.19 0)
 			(effects
