File: hardware/pcb/OpenNav_Windsensor.kicad_sch (KiCad schematic)
At the start: 11 parts, among them IC1 AS5600-ASOT, J1 Conn_01x02_Pin, U1 XIAO-ESP32-C6, U2 StpDwnE3.3-0.5, U3 SS411P, U4 DS18B20

Commit message: V1
Parts:
- removed C1: 10uF/50V, symbol Device:C
- removed C2: 20uF/10V, symbol Device:C
- C3: footprint (none) -> Capacitor_THT:C_Radial_D6.3mm_H11.0mm_P2.50mm
- J1: footprint (none) -> Connector_JST:JST_XH_B2B-XH-A_1x02_P2.50mm_Vertical
- R1, R2: footprint (none) -> Resistor_THT:R_Axial_DIN0207_L6.3mm_D2.5mm_P7.62mm_Horizontal
- U2: footprint Converter_DCDC:Converter_DCDC_RECOM_R-78E-0.5_THT -> Custom:CONV_R-78K3.3-0.5
- U3: footprint Package_TO_SOT_THT:TO-92Flat -> Custom:SS411P
Connections:
- net at U1.1 (GPIO0/A0/D0): now also U3.3 (V_{OUT})
- net at U1.10 (GPIO20/D9/MISO): no longer U3.3 (V_{OUT})
- net at U1.11 (GPIO18/D10/MOSI): now also U4.2 (DQ)
- net at U1.8 (GPIO17/D7/RX): no longer U4.2 (DQ)
Other:
- moved on the sheet: R2

Commit message: V2
Parts:
- C3: footprint Capacitor_THT:C_Radial_D6.3mm_H11.0mm_P2.50mm -> Capacitor_THT:C_Disc_D8.0mm_W5.0mm_P7.50mm
Connections:
- net at U1.1 (GPIO0/A0/D0): no longer U3.3 (V_{OUT})
- net at U1.7 (GPIO16/D6/TX): now also U3.3 (V_{OUT})
Changed lines of the file:
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@@
+	)
+	(no_connect
+		(at 125.73 104.14)
 	)
 	(no_connect
@@
 	)
 	(no_connect
-		(at 125.73 127)
-	)
-	(no_connect
 		(at 113.03 125.73)
 	)
@@
 	(wire
 		(pts
+			(xy 124.46 127) (xy 125.73 127)
+		)
+		(stroke
+			(width 0)
+			(type default)
+		)
+	)
+	(wire
+		(pts
 			(xy 78.74 125.73) (xy 78.74 129.54)
 		)
@@
 	(wire
 		(pts
-			(xy 137.16 85.09) (xy 125.73 85.09)
-		)
-		(stroke
-			(width 0)
-			(type default)
-		)
-	)
-	(wire
-		(pts
 			(xy 118.11 128.27) (xy 120.65 128.27)
 		)
@@
 	(wire
 		(pts
-			(xy 125.73 85.09) (xy 125.73 104.14)
+			(xy 124.46 85.09) (xy 137.16 85.09)
+		)
+		(stroke
+			(width 0)
+			(type default)
+		)
+	)
+	(wire
+		(pts
+			(xy 124.46 85.09) (xy 124.46 127)
 		)
 		(stroke
@@
 			)
 		)
-		(property "Footprint" "Capacitor_THT:C_Radial_D6.3mm_H11.0mm_P2.50mm"
+		(property "Footprint" "Capacitor_THT:C_Disc_D8.0mm_W5.0mm_P7.50mm"
 			(at 78.74 123.19 0)
 			(effects

Commit message: Corrected capacitor size based on what bought
Parts:
- C3: footprint Capacitor_THT:C_Disc_D8.0mm_W5.0mm_P7.50mm -> Capacitor_THT:C_Disc_D7.5mm_W5.0mm_P10.00mm
Changed lines of the file:
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@@
 			)
 		)
-		(property "Footprint" "Capacitor_THT:C_Disc_D8.0mm_W5.0mm_P7.50mm"
+		(property "Footprint" "Capacitor_THT:C_Disc_D7.5mm_W5.0mm_P10.00mm"
 			(at 78.74 123.19 0)
 			(effects
